Commit message: Adding the 4th link to the arm_4DOF.urdf model

File: my_armsim/urdf/arm_4DOF.urdf (robot description, URDF)
Before this commit: robot visual, 4 links, 3 joints
Links:
- added link link4; visual cylinder length=0.02 radius=0.02
- link link1: geometry visual cylinder length=0.08 radius=0.02
Joints:
- added joint link3_to_link4: type revolute, parent link3, child link4, origin xyz=0.2 0.0 0.0 rpy=0 -0.7 0, axis 0 0 1, limit lower=-1.5 upper=1.5 effort=1000.0 velocity=0.5
- joint link1_to_link2: origin xyz=0.0 0.0 0.06 rpy=0 0 0 -> xyz=0.0 0.0 0.07 rpy=0 0 0
